Commit message: wip

File: description/gazebo_control copy.xacro (robot description, xacro)
@@ -4,7 +4,12 @@
     <gazebo>
         <plugin name="diff_drive" filename="libgazebo_ros_diff_drive.so">
+            <ros>
+                <namespace>${robot_namespace}</namespace>
+                <argument>cmd_vel:=${robot_namespace}/cmd_vel</argument>
+                <argument>odom:=${robot_namespace}/odom</argument>
+            </ros>
             <!-- Wheel Information -->
-            <left_joint>left_wheel_joint</left_joint>
-            <right_joint>right_wheel_joint</right_joint>
+            <left_joint>${robot_namespace}/left_wheel_joint</left_joint>
+            <right_joint>${robot_namespace}/right_wheel_joint</right_joint>
             <wheel_separation>0.297</wheel_separation>
             <wheel_diameter>0.066</wheel_diameter>
@@ -13,6 +18,6 @@
             <max_wheel_acceleration>10.0</max_wheel_acceleration>
             <!-- Output -->
-            <odometry_frame>odom</odometry_frame>
-            <robot_base_frame>base_link</robot_base_frame>
+            <odometry_frame>${robot_namespace}/odom</odometry_frame>
+            <robot_base_frame>${robot_namespace}/base_link</robot_base_frame>
             <publish_odom>true</publish_odom>
             <publish_odom_tf>true</publish_odom_tf>

File: description/lidar copy.xacro (robot description, xacro)
@@ -1,10 +1,10 @@
 <?xml version="1.0"?>
 <robot xmlns:xacro="http://www.ros.org/wiki/xacro" >
-    <joint name="laser_joint" type="fixed">
-        <parent link="chassis"/>
-        <child link="laser_frame"/>
+    <joint name="${robot_namespace}/laser_joint" type="fixed">
+        <parent link="${robot_namespace}/chassis"/>
+        <child link="${robot_namespace}/laser_frame"/>
         <origin xyz="0.122 0 0.212" rpy="0 0 0"/>
     </joint>
-    <link name="laser_frame">
+    <link name="${robot_namespace}/laser_frame">
         <visual>
             <geometry>
@@ -29,5 +29,5 @@
         </xacro:inertial_cylinder>
     </link>
-    <gazebo reference="laser_frame">
+    <gazebo reference="${robot_namespace}/laser_frame">
         <material>Gazebo/Black</material>
         <sensor name="laser" type="ray">
@@ -50,9 +50,9 @@
             <plugin name="laser_controller" filename="libgazebo_ros_ray_sensor.so">
                 <ros>
-                    <namespace></namespace>
-                    <remapping>~/out:=laserscan</remapping>
+                    <namespace>${robot_namespace}</namespace>
+                    <argument>~/out:=scan</argument>
                 </ros>
                 <output_type>sensor_msgs/LaserScan</output_type>
-                <frame_name>laser_frame</frame_name>
+                <frame_name>${robot_namespace}/laser_frame</frame_name>
             </plugin>
         </sensor>

File: description/robot.urdf copy.xacro (robot description, xacro)
@@ -1,5 +1,5 @@
 <?xml version="1.0"?>
 <robot xmlns:xacro="http://www.ros.org/wiki/xacro"  name="robot">
-    <xacro:arg name="robot_ns" default="eigen0"/>
+    <xacro:arg name="robot_ns" default=""/>
     <xacro:property name="robot_namespace" value="$(arg robot_ns)"/>
     <xacro:arg name="use_ros2_control" default="true"/>

File: description/robot_core copy.xacro (robot description, xacro)
@@ -34,21 +34,21 @@
     </material>
     <!-- BASE LINK -->
-    <link name="base_link">
+    <link name="${robot_namespace}/base_link">
     </link>
     <!-- BASE_FOOTPRINT LINK -->
-    <joint name="base_footprint_joint" type="fixed">
-        <parent link="base_link"/>
-        <child link="base_footprint"/>
+    <joint name="${robot_namespace}/base_footprint_joint" type="fixed">
+        <parent link="${robot_namespace}/base_link"/>
+        <child link="${robot_namespace}/base_footprint"/>
         <origin xyz="0 0 0" rpy="0 0 0"/>
     </joint>
-    <link name="base_footprint">
+    <link name="${robot_namespace}/base_footprint">
     </link>
     <!-- CHASSIS LINK -->
-    <joint name="chassis_joint" type="fixed">
-        <parent link="base_link"/>
-        <child link="chassis"/>
+    <joint name="${robot_namespace}/chassis_joint" type="fixed">
+        <parent link="${robot_namespace}/base_link"/>
+        <child link="${robot_namespace}/chassis"/>
         <origin xyz="${-wheel_offset_x} 0 ${-wheel_offset_z}"/>
     </joint>
-    <link name="chassis">
+    <link name="${robot_namespace}/chassis">
         <visual>
             <origin xyz="${chassis_length/2} 0 ${chassis_height/2}"/>
@@ -68,15 +68,15 @@
         </xacro:inertial_box>
     </link>
-    <gazebo reference="chassis">
+    <gazebo reference="${robot_namespace}/chassis">
         <material>Gazebo/Orange</material>
     </gazebo>
     <!-- LEFT WHEEL LINK -->
-    <joint name="left_wheel_joint" type="continuous">
-        <parent link="base_link"/>
-        <child link="left_wheel"/>
+    <joint name="${robot_namespace}/left_wheel_joint" type="continuous">
+        <parent link="${robot_namespace}/base_link"/>
+        <child link="${robot_namespace}/left_wheel"/>
         <origin xyz="0 ${wheel_offset_y} 0" rpy="-${pi/2} 0 0" />
         <axis xyz="0 0 1"/>
     </joint>
-    <link name="left_wheel">
+    <link name="${robot_namespace}/left_wheel">
         <visual>
             <geometry>
@@ -94,15 +94,15 @@
         </xacro:inertial_cylinder>
     </link>
-    <gazebo reference="left_wheel">
+    <gazebo reference="${robot_namespace}/left_wheel">
         <material>Gazebo/Blue</material>
     </gazebo>
     <!-- RIGHT WHEEL LINK -->
-    <joint name="right_wheel_joint" type="continuous">
-        <parent link="base_link"/>
-        <child link="right_wheel"/>
+    <joint name="${robot_namespace}/right_wheel_joint" type="continuous">
+        <parent link="${robot_namespace}/base_link"/>
+        <child link="${robot_namespace}/right_wheel"/>
         <origin xyz="0 ${-wheel_offset_y} 0" rpy="${pi/2} 0 0" />
         <axis xyz="0 0 -1"/>
     </joint>
-    <link name="right_wheel">
+    <link name="${robot_namespace}/right_wheel">
         <visual>
             <geometry>
@@ -120,14 +120,14 @@
         </xacro:inertial_cylinder>
     </link>
-    <gazebo reference="right_wheel">
+    <gazebo reference="${robot_namespace}/right_wheel">
         <material>Gazebo/Blue</material>
     </gazebo>
     <!-- CASTER WHEEL LINK -->
-    <joint name="caster_wheel_joint" type="fixed">
-        <parent link="chassis"/>
-        <child link="caster_wheel"/>
+    <joint name="${robot_namespace}/caster_wheel_joint" type="fixed">
+        <parent link="${robot_namespace}/chassis"/>
+        <child link="${robot_namespace}/caster_wheel"/>
         <origin xyz="${caster_wheel_offset_x} 0 ${caster_wheel_offset_z}"/>
     </joint>
-    <link name="caster_wheel">
+    <link name="${robot_namespace}/caster_wheel">
         <visual>
             <geometry>
@@ -145,5 +145,5 @@
         </xacro:inertial_sphere>
     </link>
-    <gazebo reference="caster_wheel">
+    <gazebo reference="${robot_namespace}/caster_wheel">
         <material>Gazebo/White</material>
         <mu1 value="0.001"/>

File: description/ros2_control copy.xacro (robot description, xacro)
@@ -14,5 +14,5 @@
                 <param name="enc_counts_per_rev">3436</param>
             </hardware>
-            <joint name="left_wheel_joint">
+            <joint name="${robot_namespace}/left_wheel_joint">
                 <command_interface name="velocity">
                     <param name="min">-10</param>
@@ -22,5 +22,5 @@
                 <state_interface name="position"/>
             </joint>
-            <joint name="right_wheel_joint">
+            <joint name="${robot_namespace}/right_wheel_joint">
                 <command_interface name="velocity">
                     <param name="min">-10</param>
@@ -37,5 +37,5 @@
                 <plugin>gazebo_ros2_control/GazeboSystem</plugin>
             </hardware>
-            <joint name="left_wheel_joint">
+            <joint name="${robot_namespace}/left_wheel_joint">
                 <command_interface name="velocity">
                     <param name="min">-10</param>
@@ -45,5 +45,5 @@
                 <state_interface name="position"/>
             </joint>
-            <joint name="right_wheel_joint">
+            <joint name="${robot_namespace}/right_wheel_joint">
                 <command_interface name="velocity">
                     <param name="min">-10</param>
